Commit message: [WIP]create packages

File: mfja_motoman_hc10/urdf/hc10dt_b10.xacro (robot description, xacro)
@@ -1,5 +1,5 @@
 <?xml version="1.0" ?>
 <robot name="motoman_hc10dt_b10" xmlns:xacro="http://ros.org/wiki/xacro">
-  <xacro:include filename="$(find motoman_hc10_moveit_config)/urdf/hc10dt_b10_macro.xacro" />
+  <xacro:include filename="$(find mfja_motoman_hc10)/urdf/hc10dt_b10_macro.xacro" />
   <xacro:motoman_hc10dt_b10 prefix="yaska1_"/>
 </robot>

File: mfja_motoman_hc10/urdf/left/cell.xacro (robot description, xacro)
@@ -5,5 +5,5 @@
       <origin rpy="0 0 0" xyz="0 0 0"/>
       <geometry>
-        <mesh filename="package://motoman_hc10_moveit_config/meshes/env/pieds_cellule.stl" scale="1 1 1"/>
+        <mesh filename="package://mfja_motoman_hc10/meshes/env/pieds_cellule.stl" scale="1 1 1"/>
       </geometry>
       <material name="silver"/>
@@ -12,5 +12,5 @@
       <origin rpy="0 0 0" xyz="0 0 0"/>
       <geometry>
-        <mesh filename="package://motoman_hc10_moveit_config/meshes/env/pieds_cellule.stl" scale="1 1 1"/>
+        <mesh filename="package://mfja_motoman_hc10/meshes/env/pieds_cellule.stl" scale="1 1 1"/>
       </geometry>
     </collision>
@@ -20,5 +20,5 @@
       <origin rpy="0 0 0" xyz="0 0 0"/>
       <geometry>
-        <mesh filename="package://motoman_hc10_moveit_config/meshes/env/ergots.stl" scale="0.001 0.001 0.001"/>
+        <mesh filename="package://mfja_motoman_hc10/meshes/env/ergots.stl" scale="0.001 0.001 0.001"/>
       </geometry>
       <material name="dark_gray"/>
@@ -27,5 +27,5 @@
       <origin rpy="0 0 0" xyz="0 0 0"/>
       <geometry>
-        <mesh filename="package://motoman_hc10_moveit_config/meshes/env/ergots.stl" scale="0.001 0.001 0.001"/>
+        <mesh filename="package://mfja_motoman_hc10/meshes/env/ergots.stl" scale="0.001 0.001 0.001"/>
       </geometry>
     </collision>
@@ -35,5 +35,5 @@
       <origin rpy="0 0 0" xyz="0 0 0"/>
       <geometry>
-        <mesh filename="package://motoman_hc10_moveit_config/meshes/env/ergots.stl" scale="0.001 0.001 0.001"/>
+        <mesh filename="package://mfja_motoman_hc10/meshes/env/ergots.stl" scale="0.001 0.001 0.001"/>
       </geometry>
       <material name="dark_gray"/>
@@ -42,5 +42,5 @@
       <origin rpy="0 0 0" xyz="0 0 0"/>
       <geometry>
-        <mesh filename="package://motoman_hc10_moveit_config/meshes/env/ergots.stl" scale="0.001 0.001 0.001"/>
+        <mesh filename="package://mfja_motoman_hc10/meshes/env/ergots.stl" scale="0.001 0.001 0.001"/>
       </geometry>
     </collision>
@@ -50,5 +50,5 @@
       <origin rpy="0 0 0" xyz="0 0 0"/>
       <geometry>
-        <mesh filename="package://motoman_hc10_moveit_config/meshes/env/rail_milieu.stl" scale="0.001 0.001 0.001"/>
+        <mesh filename="package://mfja_motoman_hc10/meshes/env/rail_milieu.stl" scale="0.001 0.001 0.001"/>
       </geometry>
       <material name="silver"/>
@@ -57,5 +57,5 @@
       <origin rpy="0 0 0" xyz="0 0 0"/>
       <geometry>
-        <mesh filename="package://motoman_hc10_moveit_config/meshes/env/rail_milieu.stl" scale="0.001 0.001 0.001"/>
+        <mesh filename="package://mfja_motoman_hc10/meshes/env/rail_milieu.stl" scale="0.001 0.001 0.001"/>
       </geometry>
     </collision>
@@ -65,5 +65,5 @@
       <origin rpy="0 0 0" xyz="0 0 0"/>
       <geometry>
-        <mesh filename="package://motoman_hc10_moveit_config/meshes/env/rail_tournant.stl" scale="0.001 0.001 0.001"/>
+        <mesh filename="package://mfja_motoman_hc10/meshes/env/rail_tournant.stl" scale="0.001 0.001 0.001"/>
       </geometry>
       <material name="silver"/>
@@ -72,5 +72,5 @@
       <origin rpy="0 0 0" xyz="0 0 0"/>
       <geometry>
-        <mesh filename="package://motoman_hc10_moveit_config/meshes/env/rail_tournant.stl" scale="0.001 0.001 0.001"/>
+        <mesh filename="package://mfja_motoman_hc10/meshes/env/rail_tournant.stl" scale="0.001 0.001 0.001"/>
       </geometry>
     </collision>
@@ -80,5 +80,5 @@
       <origin rpy="0 0 0" xyz="0 0 0"/>
       <geometry>
-        <mesh filename="package://motoman_hc10_moveit_config/meshes/env/rail_tournant.stl" scale="0.001 0.001 0.001"/>
+        <mesh filename="package://mfja_motoman_hc10/meshes/env/rail_tournant.stl" scale="0.001 0.001 0.001"/>
       </geometry>
       <material name="silver"/>
@@ -87,5 +87,5 @@
       <origin rpy="0 0 0" xyz="0 0 0"/>
       <geometry>
-        <mesh filename="package://motoman_hc10_moveit_config/meshes/env/rail_tournant.stl" scale="0.001 0.001 0.001"/>
+        <mesh filename="package://mfja_motoman_hc10/meshes/env/rail_tournant.stl" scale="0.001 0.001 0.001"/>
       </geometry>
     </collision>

File: mfja_motoman_hc10/urdf/left/hc10dt_with_env.xacro (robot description, xacro)
@@ -2,9 +2,9 @@
 <robot name="yaskawa_L" xmlns:xacro="http://www.ros.org/wiki/xacro" >
     <!-- loading urdf -->
-    <xacro:include filename="$(find motoman_hc10_moveit_config)/urdf/materials.xacro" />
-    <xacro:include filename="$(find motoman_hc10_moveit_config)/urdf/table.xacro" />
-    <xacro:include filename="$(find motoman_hc10_moveit_config)/urdf/left/cell.xacro" />
-    <xacro:include filename="$(find motoman_hc10_moveit_config)/urdf/left/pince.xacro" />
-    <xacro:include filename="$(find motoman_hc10_moveit_config)/urdf/hc10dt_b10_macro.xacro" />
+    <xacro:include filename="$(find mfja_motoman_hc10)/urdf/materials.xacro" />
+    <xacro:include filename="$(find mfja_motoman_hc10)/urdf/table.xacro" />
+    <xacro:include filename="$(find mfja_motoman_hc10)/urdf/left/cell.xacro" />
+    <xacro:include filename="$(find mfja_motoman_hc10)/urdf/left/pince.xacro" />
+    <xacro:include filename="$(find motoman_hc10_support)/urdf/hc10dt_b10_macro.xacro" />
     <xacro:motoman_hc10dt_b10 prefix=""/>
     <!-- linking robot to world,workspaces and end-effector -->

File: mfja_motoman_hc10/urdf/left/pince.xacro (robot description, xacro)
@@ -5,5 +5,5 @@
       <visual>
         <geometry>
-          <mesh filename="package://motoman_hc10_moveit_config/meshes/hand/left/LWR50F-17-04-A.stl" scale="0.001 0.001 0.001"/>
+          <mesh filename="package://mfja_motoman_hc10/meshes/hand/left/LWR50F-17-04-A.stl" scale="0.001 0.001 0.001"/>
         </geometry>
         <material name="dark_gray"/>
@@ -11,5 +11,5 @@
       <collision>
         <geometry>
-          <mesh filename="package://motoman_hc10_moveit_config/meshes/hand/left/LWR50F-17-04-A.stl" scale="0.001 0.001 0.001"/>
+          <mesh filename="package://mfja_motoman_hc10/meshes/hand/left/LWR50F-17-04-A.stl" scale="0.001 0.001 0.001"/>
         </geometry>
       </collision>
@@ -18,5 +18,5 @@
       <visual>
         <geometry>
-          <mesh filename="package://motoman_hc10_moveit_config/meshes/hand/left/end_effector_LWR50L-03-00001-A.stl" scale="0.001 0.001 0.001"/>
+          <mesh filename="package://mfja_motoman_hc10/meshes/hand/left/end_effector_LWR50L-03-00001-A.stl" scale="0.001 0.001 0.001"/>
         </geometry>
         <material name="white_smoke"/>
@@ -24,5 +24,5 @@
       <collision>
         <geometry>
-          <mesh filename="package://motoman_hc10_moveit_config/meshes/hand/left/end_effector_LWR50L-03-00001-A.stl" scale="0.001 0.001 0.001"/>
+          <mesh filename="package://mfja_motoman_hc10/meshes/hand/left/end_effector_LWR50L-03-00001-A.stl" scale="0.001 0.001 0.001"/>
         </geometry>
       </collision>
@@ -31,5 +31,5 @@
         <visual>
           <geometry>
-            <mesh filename="package://motoman_hc10_moveit_config/meshes/hand/left/mors_for_LWR50L-03-00001-A.stl" scale="0.001 0.001 0.001"/>
+            <mesh filename="package://mfja_motoman_hc10/meshes/hand/left/mors_for_LWR50L-03-00001-A.stl" scale="0.001 0.001 0.001"/>
           </geometry>
           <material name="silver"/>
@@ -37,5 +37,5 @@
         <collision>
           <geometry>
-            <mesh filename="package://motoman_hc10_moveit_config/meshes/hand/left/mors_for_LWR50L-03-00001-A.stl" scale="0.001 0.001 0.001"/>
+            <mesh filename="package://mfja_motoman_hc10/meshes/hand/left/mors_for_LWR50L-03-00001-A.stl" scale="0.001 0.001 0.001"/>
           </geometry>
         </collision>
@@ -44,5 +44,5 @@
         <visual>
           <geometry>
-            <mesh filename="package://motoman_hc10_moveit_config/meshes/hand/left/mors_for_LWR50L-03-00001-A.stl" scale="0.001 0.001 0.001"/>
+            <mesh filename="package://mfja_motoman_hc10/meshes/hand/left/mors_for_LWR50L-03-00001-A.stl" scale="0.001 0.001 0.001"/>
           </geometry>
           <material name="silver"/>
@@ -50,5 +50,5 @@
         <collision>
           <geometry>
-            <mesh filename="package://motoman_hc10_moveit_config/meshes/hand/left/mors_for_LWR50L-03-00001-A.stl" scale="0.001 0.001 0.001"/>
+            <mesh filename="package://mfja_motoman_hc10/meshes/hand/left/mors_for_LWR50L-03-00001-A.stl" scale="0.001 0.001 0.001"/>
           </geometry>
         </collision>

File: mfja_motoman_hc10/urdf/right/hc10_with_env.xacro (robot description, xacro)
@@ -2,8 +2,8 @@
 <robot name="yaskawa_R" xmlns:xacro="http://www.ros.org/wiki/xacro" >
     <!-- loading urdf -->
-    <xacro:include filename="$(find motoman_hc10_moveit_config)/urdf/materials.xacro" />
-    <xacro:include filename="$(find motoman_hc10_moveit_config)/urdf/table.xacro" />
-    <xacro:include filename="$(find motoman_hc10_moveit_config)/urdf/right/cell.xacro" />
-    <xacro:include filename="$(find motoman_hc10_moveit_config)/urdf/right/pince.xacro" />
+    <xacro:include filename="$(find mfja_motoman_hc10)/urdf/materials.xacro" />
+    <xacro:include filename="$(find mfja_motoman_hc10)/urdf/table.xacro" />
+    <xacro:include filename="$(find mfja_motoman_hc10)/urdf/right/cell.xacro" />
+    <xacro:include filename="$(find mfja_motoman_hc10)/urdf/right/pince.xacro" />
     <xacro:include filename="$(find motoman_hc10_support)/urdf/hc10_macro.xacro" />
     <xacro:motoman_hc10 prefix=""/>

File: mfja_motoman_hc10/urdf/right/pince.xacro (robot description, xacro)
@@ -5,5 +5,5 @@
       <visual>
         <geometry>
-          <mesh filename="package://motoman_hc10_moveit_config/meshes/hand/right/cylinder.stl" scale="1 1 1"/>
+          <mesh filename="package://mfja_motoman_hc10/meshes/hand/right/cylinder.stl" scale="1 1 1"/>
         </geometry>
         <material name="white_smoke"/>
@@ -11,5 +11,5 @@
       <collision>
         <geometry>
-          <mesh filename="package://motoman_hc10_moveit_config/meshes/hand/right/cylinder.stl" scale="1 1 1"/>
+          <mesh filename="package://mfja_motoman_hc10/meshes/hand/right/cylinder.stl" scale="1 1 1"/>
         </geometry>
       </collision>
@@ -18,5 +18,5 @@
         <visual>
           <geometry>
-            <mesh filename="package://motoman_hc10_moveit_config/meshes/hand/right/GEH6040IL-03-B(01).stl" scale="0.001 0.001 0.001"/>
+            <mesh filename="package://mfja_motoman_hc10/meshes/hand/right/GEH6040IL-03-B(01).stl" scale="0.001 0.001 0.001"/>
           </geometry>
           <material name="dark_gray"/>
@@ -24,5 +24,5 @@
         <collision>
           <geometry>
-            <mesh filename="package://motoman_hc10_moveit_config/meshes/hand/right/GEH6040IL-03-B(01).stl" scale="0.001 0.001 0.001"/>
+            <mesh filename="package://mfja_motoman_hc10/meshes/hand/right/GEH6040IL-03-B(01).stl" scale="0.001 0.001 0.001"/>
           </geometry>
         </collision>
@@ -31,5 +31,5 @@
         <visual>
           <geometry>
-            <mesh filename="package://motoman_hc10_moveit_config/meshes/hand/right/UB5006AL.stl" scale="0.001 0.001 0.001"/>
+            <mesh filename="package://mfja_motoman_hc10/meshes/hand/right/UB5006AL.stl" scale="0.001 0.001 0.001"/>
           </geometry>
           <material name="silver"/>
@@ -37,5 +37,5 @@
         <collision>
           <geometry>
-            <mesh filename="package://motoman_hc10_moveit_config/meshes/hand/right/UB5006AL.stl" scale="0.001 0.001 0.001"/>
+            <mesh filename="package://mfja_motoman_hc10/meshes/hand/right/UB5006AL.stl" scale="0.001 0.001 0.001"/>
           </geometry>
         </collision>
@@ -44,5 +44,5 @@
         <visual>
           <geometry>
-            <mesh filename="package://motoman_hc10_moveit_config/meshes/hand/right/UB5006AL.stl" scale="0.001 0.001 0.001"/>
+            <mesh filename="package://mfja_motoman_hc10/meshes/hand/right/UB5006AL.stl" scale="0.001 0.001 0.001"/>
           </geometry>
           <material name="silver"/>
@@ -50,5 +50,5 @@
         <collision>
           <geometry>
-            <mesh filename="package://motoman_hc10_moveit_config/meshes/hand/right/UB5006AL.stl" scale="0.001 0.001 0.001"/>
+            <mesh filename="package://mfja_motoman_hc10/meshes/hand/right/UB5006AL.stl" scale="0.001 0.001 0.001"/>
           </geometry>
         </collision>
@@ -57,5 +57,5 @@
         <visual>
           <geometry>
-            <mesh filename="package://motoman_hc10_moveit_config/meshes/hand/right/APR000009.stl" scale="0.001 0.001 0.001"/>
+            <mesh filename="package://mfja_motoman_hc10/meshes/hand/right/APR000009.stl" scale="0.001 0.001 0.001"/>
           </geometry>
           <material name="dark_gray"/>
@@ -63,5 +63,5 @@
         <collision>
           <geometry>
-            <mesh filename="package://motoman_hc10_moveit_config/meshes/hand/right/APR000009.stl" scale="0.001 0.001 0.001"/>
+            <mesh filename="package://mfja_motoman_hc10/meshes/hand/right/APR000009.stl" scale="0.001 0.001 0.001"/>
           </geometry>
         </collision>
@@ -70,5 +70,5 @@
         <visual>
           <geometry>
-            <mesh filename="package://motoman_hc10_moveit_config/meshes/hand/right/APGEH6000.stl" scale="0.001 0.001 0.001"/>
+            <mesh filename="package://mfja_motoman_hc10/meshes/hand/right/APGEH6000.stl" scale="0.001 0.001 0.001"/>
           </geometry>
           <material name="dark_gray"/>
@@ -76,5 +76,5 @@
         <collision>
           <geometry>
-            <mesh filename="package://motoman_hc10_moveit_config/meshes/hand/right/APGEH6000.stl" scale="0.001 0.001 0.001"/>
+            <mesh filename="package://mfja_motoman_hc10/meshes/hand/right/APGEH6000.stl" scale="0.001 0.001 0.001"/>
           </geometry>
         </collision>
@@ -83,5 +83,5 @@
         <visual>
           <geometry>
-            <mesh filename="package://motoman_hc10_moveit_config/meshes/hand/right/APGEH6000.stl" scale="0.001 0.001 0.001"/>
+            <mesh filename="package://mfja_motoman_hc10/meshes/hand/right/APGEH6000.stl" scale="0.001 0.001 0.001"/>
           </geometry>
           <material name="dark_gray"/>
@@ -89,5 +89,5 @@
         <collision>
           <geometry>
-            <mesh filename="package://motoman_hc10_moveit_config/meshes/hand/right/APGEH6000.stl" scale="0.001 0.001 0.001"/>
+            <mesh filename="package://mfja_motoman_hc10/meshes/hand/right/APGEH6000.stl" scale="0.001 0.001 0.001"/>
           </geometry>
         </collision>

File: mfja_motoman_hc10/urdf/table.xacro (robot description, xacro)
@@ -5,5 +5,5 @@
       <origin rpy="0 0 0" xyz="0 0 0"/>
       <geometry>
-        <mesh filename="package://motoman_hc10_moveit_config/meshes/env/table_yaskawa.stl" scale="1 1 1"/>
+        <mesh filename="package://mfja_motoman_hc10/meshes/env/table_yaskawa.stl" scale="1 1 1"/>
       </geometry>
       <material name="silver"/>
@@ -12,5 +12,5 @@
       <origin rpy="0 0 0" xyz="0 0 0"/>
       <geometry>
-        <mesh filename="package://motoman_hc10_moveit_config/meshes/env/table_yaskawa.stl" scale="1 1 1"/>
+        <mesh filename="package://mfja_motoman_hc10/meshes/env/table_yaskawa.stl" scale="1 1 1"/>
       </geometry>
     </collision>
