Commit message: First working version on real robot

File: mfja_motoman_hc10/urdf/left/hc10dt_with_env.xacro (robot description, xacro)
@@ -21,5 +21,5 @@
     </joint>
     <joint name="table_joint" type="fixed">
-        <origin rpy="-1.57079 1.57079 0" xyz="0.171 0.203 0.181" />
+        <origin rpy="-1.57079 3.1415 0" xyz="0.171 0.203 0.181" />
         <parent link="table_link" />
         <child link="base_link" />

File: mfja_motoman_hc10/urdf/right/cell.xacro (robot description, xacro)
@@ -5,5 +5,5 @@
       <origin rpy="0 0 0" xyz="0 0 0"/>
       <geometry>
-        <mesh filename="package://motoman_hc10_moveit_config/meshes/env/pieds_cellule.stl" scale="1 1 1"/>
+        <mesh filename="package://mfja_motoman_hc10/meshes/env/pieds_cellule.stl" scale="1 1 1"/>
       </geometry>
       <material name="silver"/>
@@ -12,5 +12,5 @@
       <origin rpy="0 0 0" xyz="0 0 0"/>
       <geometry>
-        <mesh filename="package://motoman_hc10_moveit_config/meshes/env/pieds_cellule.stl" scale="1 1 1"/>
+        <mesh filename="package://mfja_motoman_hc10/meshes/env/pieds_cellule.stl" scale="1 1 1"/>
       </geometry>
     </collision>
@@ -20,5 +20,5 @@
       <origin rpy="0 0 0" xyz="0 0 0"/>
       <geometry>
-        <mesh filename="package://motoman_hc10_moveit_config/meshes/env/ergots.stl" scale="0.001 0.001 0.001"/>
+        <mesh filename="package://mfja_motoman_hc10/meshes/env/ergots.stl" scale="0.001 0.001 0.001"/>
       </geometry>
       <material name="dark_gray"/>
@@ -27,5 +27,5 @@
       <origin rpy="0 0 0" xyz="0 0 0"/>
       <geometry>
-        <mesh filename="package://motoman_hc10_moveit_config/meshes/env/ergots.stl" scale="0.001 0.001 0.001"/>
+        <mesh filename="package://mfja_motoman_hc10/meshes/env/ergots.stl" scale="0.001 0.001 0.001"/>
       </geometry>
     </collision>
@@ -35,5 +35,5 @@
       <origin rpy="0 0 0" xyz="0 0 0"/>
       <geometry>
-        <mesh filename="package://motoman_hc10_moveit_config/meshes/env/ergots.stl" scale="0.001 0.001 0.001"/>
+        <mesh filename="package://mfja_motoman_hc10/meshes/env/ergots.stl" scale="0.001 0.001 0.001"/>
       </geometry>
       <material name="dark_gray"/>
@@ -42,5 +42,5 @@
       <origin rpy="0 0 0" xyz="0 0 0"/>
       <geometry>
-        <mesh filename="package://motoman_hc10_moveit_config/meshes/env/ergots.stl" scale="0.001 0.001 0.001"/>
+        <mesh filename="package://mfja_motoman_hc10/meshes/env/ergots.stl" scale="0.001 0.001 0.001"/>
       </geometry>
     </collision>
@@ -50,5 +50,5 @@
       <origin rpy="0 0 0" xyz="0 0 0"/>
       <geometry>
-        <mesh filename="package://motoman_hc10_moveit_config/meshes/env/rail_milieu.stl" scale="0.001 0.001 0.001"/>
+        <mesh filename="package://mfja_motoman_hc10/meshes/env/rail_milieu.stl" scale="0.001 0.001 0.001"/>
       </geometry>
       <material name="silver"/>
@@ -57,5 +57,5 @@
       <origin rpy="0 0 0" xyz="0 0 0"/>
       <geometry>
-        <mesh filename="package://motoman_hc10_moveit_config/meshes/env/rail_milieu.stl" scale="0.001 0.001 0.001"/>
+        <mesh filename="package://mfja_motoman_hc10/meshes/env/rail_milieu.stl" scale="0.001 0.001 0.001"/>
       </geometry>
     </collision>
@@ -65,5 +65,5 @@
       <origin rpy="0 0 0" xyz="0 0 0"/>
       <geometry>
-        <mesh filename="package://motoman_hc10_moveit_config/meshes/env/rail_tournant.stl" scale="0.001 0.001 0.001"/>
+        <mesh filename="package://mfja_motoman_hc10/meshes/env/rail_tournant.stl" scale="0.001 0.001 0.001"/>
       </geometry>
       <material name="silver"/>
@@ -72,5 +72,5 @@
       <origin rpy="0 0 0" xyz="0 0 0"/>
       <geometry>
-        <mesh filename="package://motoman_hc10_moveit_config/meshes/env/rail_tournant.stl" scale="0.001 0.001 0.001"/>
+        <mesh filename="package://mfja_motoman_hc10/meshes/env/rail_tournant.stl" scale="0.001 0.001 0.001"/>
       </geometry>
     </collision>
@@ -80,5 +80,5 @@
       <origin rpy="0 0 0" xyz="0 0 0"/>
       <geometry>
-        <mesh filename="package://motoman_hc10_moveit_config/meshes/env/rail_tournant.stl" scale="0.001 0.001 0.001"/>
+        <mesh filename="package://mfja_motoman_hc10/meshes/env/rail_tournant.stl" scale="0.001 0.001 0.001"/>
       </geometry>
       <material name="silver"/>
@@ -87,5 +87,5 @@
       <origin rpy="0 0 0" xyz="0 0 0"/>
       <geometry>
-        <mesh filename="package://motoman_hc10_moveit_config/meshes/env/rail_tournant.stl" scale="0.001 0.001 0.001"/>
+        <mesh filename="package://mfja_motoman_hc10/meshes/env/rail_tournant.stl" scale="0.001 0.001 0.001"/>
       </geometry>
     </collision>

File: mfja_motoman_hc10/urdf/right/hc10_with_env.xacro (robot description, xacro)
@@ -7,5 +7,5 @@
     <xacro:include filename="$(find mfja_motoman_hc10)/urdf/right/pince.xacro" />
     <xacro:include filename="$(find motoman_hc10_support)/urdf/hc10_macro.xacro" />
-    <xacro:motoman_hc10 prefix="yaskawa_RIGHT_"/>
+    <xacro:motoman_hc10 prefix=""/>
     <!-- linking robot to world,workspaces and end-effector -->
     <link name="world" />
