Commit message: Control via RViz now works

File: mfja_motoman_hc10/urdf/left/pince.xacro (robot description, xacro)
@@ -61,18 +61,18 @@
       </joint>
       <!-- ce joint doit être de type prismatique -->
-      <joint name="end_effector_adaptater_mors1" type="prismatic" >
+      <joint name="end_effector_adaptater_mors1" type="fixed" >
         <origin rpy="0 0 0" xyz="0 0 0" />
         <parent link="end_effector_link" />
         <child link="mors_link1" />
-        <axis xyz="0 0 1"/>
-        <limit effort="1000.0" lower="-0.0108" upper="0" velocity="0.5"/>
+        <!-- <axis xyz="0 0 1"/> -->
+        <!-- <limit effort="1000.0" lower="-0.0108" upper="0" velocity="0.5"/> -->
       </joint>
       <!-- ce joint doit être de type prismatique -->
-      <joint name="end_effector_adaptater_mors2" type="prismatic" >
+      <joint name="end_effector_adaptater_mors2" type="fixed" >
         <origin rpy="0 3.14 0" xyz="0 0 0" />
         <parent link="end_effector_link" />
         <child link="mors_link2" />
-        <axis xyz="0 0 1"/>
-        <limit effort="1000.0" lower="-0.0108" upper="0" velocity="0.5"/>
+        <!-- <axis xyz="0 0 1"/> -->
+        <!-- <limit effort="1000.0" lower="-0.0108" upper="0" velocity="0.5"/> -->
       </joint>
 </robot>

File: mfja_motoman_hc10/urdf/right/pince.xacro (robot description, xacro)
@@ -105,16 +105,16 @@
       </joint>
       <!-- ce joint doit être de type prismatique -->
-      <joint name="end_effector_adaptater_mors1" type="prismatic" >
+      <joint name="end_effector_adaptater_mors1" type="fixed" >
         <origin rpy="3.14 0 0" xyz="-0.079 -0.045 0.006" />
         <parent link="end_effector_link" />
         <child link="adaptater_mors1_link" />
-        <limit effort="1000.0" lower="0" upper="0.035" velocity="0.5"/>
+        <!-- <limit effort="1000.0" lower="0" upper="0.035" velocity="0.5"/> -->
       </joint>
       <!-- ce joint doit être de type prismatique -->
-      <joint name="end_effector_adaptater_mors2" type="prismatic" >
+      <joint name="end_effector_adaptater_mors2" type="fixed" >
         <origin rpy="3.14 3.14 0" xyz="0.078 -0.045 -0.023" />
         <parent link="end_effector_link" />
         <child link="adaptater_mors2_link" />
-        <limit effort="1000.0" lower="0" upper="0.035" velocity="0.5"/>
+        <!-- <limit effort="1000.0" lower="0" upper="0.035" velocity="0.5"/> -->
       </joint>
       <joint name="end_effector_mors1" type="fixed" >

File: motoman_hc10_moveit_config/config/yaskawa_LEFT.ros2_control.xacro (robot description, xacro)
@@ -50,5 +50,5 @@
                 <state_interface name="velocity"/>
             </joint>
-            <joint name="end_effector_adaptater_mors1">
+            <!-- <joint name="end_effector_adaptater_mors1">
                 <command_interface name="position"/>
                 <state_interface name="position">
@@ -63,5 +63,5 @@
                 </state_interface>
                 <state_interface name="velocity"/>
-            </joint>
+            </joint> -->
         </ros2_control>
     </xacro:macro>

File: motoman_hc10_moveit_config/config/yaskawa_RIGHT.ros2_control.xacro (robot description, xacro)
@@ -50,5 +50,5 @@
                 <state_interface name="velocity"/>
             </joint>
-            <joint name="end_effector_adaptater_mors1">
+            <!-- <joint name="end_effector_adaptater_mors1">
                 <command_interface name="position"/>
                 <state_interface name="position">
@@ -63,5 +63,5 @@
                 </state_interface>
                 <state_interface name="velocity"/>
-            </joint>
+            </joint> -->
         </ros2_control>
     </xacro:macro>
